File: EduboardV2_Baseboard.kicad_pcb (KiCad board)
At the start: 2 copper layers, 100 x 160 mm, 145 parts, among them IC201 STK8321, IC202 PCF8563T_5,518, IC203 W25Q128JVSIQTR, IC301 XL1509-5.0E1, IC302 SY8113BADC, IC601 STK8321, IC602 SP3485EN-L_TR, IC603 WM8782SEDS_RV_C323842, IC604 CS4344-CZZ, IC605 MCP9700AT-E_TT, SW301 1FS1T1B9M2RES-5, SW401 K2-1102SP-C4SC-04, SW402 K2-1102SP-C4SC-04, SW403 K2-1102SP-C4SC-04, SW404 K2-1102SP-C4SC-04, T401 AO3400A, T402 AO3400A, T403 AO3400A, T404 AO3400A, T405 AO3400A, X201 PCIE-52P40H, X202 32.768 kHz, X203 TF-15×15, X301 KF2EDGR-3.81-3P, X302 USB3.1C16PFSMT, X303 CH340G, X401 ER-TFT035-6, X501 BH-00105, X502 S4B-PH-SM4-K-TB(LF)(SN), X503 USB3.1C16PFSMT, X601 KF2EDGR-3.81-3P, X602 PJ-327C-4A, X603 PJ-327C-4A, Y301 X322512MSB4SI

Commit message: slight modifications
Parts:
- moved IC203 18.4 mm to (72.0, 93.0), turned to 180 degrees
- moved B201 3.61 mm to (86.0, 71.0), turned to -90 degrees
- moved C309 3.16 mm to (85.0, 39.0)
- moved C301 3.00 mm to (89.0, 49.0)
- moved C316 2.24 mm to (77.0, 49.0)
- moved X301 2.24 mm to (71.0, 27.3)
- moved X503 2.24 mm to (88.0, 25.0)
- moved X302 2.00 mm to (105.0, 25.0)
- moved X601 2.00 mm to (138.0, 27.3)
- moved X502 1.00 mm to (121.0, 26.0)
Changed lines of the file:
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@@
     (fp_line (start -2.5 -1.91) (end -2.41 -1.91) (layer "F.SilkS") (width 0.25))
     (fp_line (start -2.5 -1.5) (end -2.5 -1.91) (layer "F.SilkS") (width 0.25))
-    (fp_arc (start -2.48726 -0.729889) (mid -2.50637 0.729972) (end -2.5 -0.73) (layer "F.SilkS") (width 0.25))
+    (fp_arc (start -2.48726 -0.729889) (mid -2.50635 0.729972) (end -2.5 -0.73) (layer "F.SilkS") (width 0.25))
     (fp_circle (center -2.54 2.67) (end -2.39 2.67) (layer "F.SilkS") (width 0.3) (fill none))
     (fp_circle (center -1.91 3.4) (end -1.76 3.4) (layer "Cmts.User") (width 0.3) (fill none))
@@
   )
   (footprint "eduboardv2:CAP-SMD_BD8.0-L8.3-W8.3-RD" (layer "F.Cu")
-    (at 78 51)
+    (at 77 49)
     (property "JLC Part" "Extended Part")
     (property "LCSC Part" "C164065")
@@
   )
   (footprint "eduboardv2:USB-C-SMD_TYPE-C-USB-17" (layer "F.Cu")
-    (at 105 27 180)
+    (at 105 25 180)
     (property "JLC Part" "Extended Part")
     (property "LCSC Part" "C167321")
@@
   )
   (footprint "eduboardv2:CONN-SMD_S4B-PH-SM4-K-TB-LF-SN" (layer "F.Cu")
-    (at 121 27)
+    (at 121 26)
     (property "JLC Part" "Extended Part")
     (property "LCSC Part" "C265332")
@@
   )
   (footprint "eduboardv2:CAP-SMD_BD8.0-L8.3-W8.3-RD" (layer "F.Cu")
-    (at 84 42 90)
+    (at 85 39 90)
     (property "JLC Part" "Extended Part")
     (property "LCSC Part" "C164065")
@@
   )
   (footprint "eduboardv2:CONN-TH_3P-P3.81_KF2EDGR-3.81-3P" (layer "F.Cu")
-    (at 137.9675 29.3325 180)
+    (at 137.9675 27.3325 180)
     (property "JLC Part" "Extended Part")
     (property "LCSC Part" "C441183")
@@
   )
   (footprint "eduboardv2:CAP-SMD_BD8.0-L8.3-W8.3-RD" (layer "F.Cu")
-    (at 89 52)
+    (at 89 49)
     (property "JLC Part" "Extended Part")
     (property "LCSC Part" "C164065")
@@
     (fp_line (start 2.5 -1.5) (end 2.5 1.5) (layer "F.SilkS") (width 0.25))
     (fp_line (start -2.5 -1.91) (end -2.41 -1.91) (layer "F.SilkS") (width 0.25))
-    (fp_arc (start -2.48726 -0.729889) (mid -2.50637 0.729972) (end -2.5 -0.73) (layer "F.SilkS") (width 0.25))
+    (fp_arc (start -2.48726 -0.729889) (mid -2.50635 0.729972) (end -2.5 -0.73) (layer "F.SilkS") (width 0.25))
     (fp_circle (center -2.54 2.67) (end -2.39 2.67) (layer "F.SilkS") (width 0.3) (fill none))
     (fp_circle (center -1.91 3.4) (end -1.76 3.4) (layer "Cmts.User") (width 0.3) (fill none))
@@
   )
   (footprint "eduboardv2:USB-C-SMD_TYPE-C-USB-17" (layer "F.Cu")
-    (at 89 27 180)
+    (at 88 25 180)
     (property "JLC Part" "Extended Part")
     (property "LCSC Part" "C167321")
@@
     (fp_line (start -2.5 -1.5) (end -2.5 -0.73) (layer "F.SilkS") (width 0.25))
     (fp_line (start 2.5 -1.5) (end 2.5 -1.91) (layer "F.SilkS") (width 0.25))
-    (fp_arc (start -2.48726 -0.729889) (mid -2.50637 0.729972) (end -2.5 -0.73) (layer "F.SilkS") (width 0.25))
+    (fp_arc (start -2.48726 -0.729889) (mid -2.50635 0.729972) (end -2.5 -0.73) (layer "F.SilkS") (width 0.25))
     (fp_circle (center -2.54 2.67) (end -2.39 2.67) (layer "F.SilkS") (width 0.3) (fill none))
     (fp_circle (center -1.91 3.4) (end -1.76 3.4) (layer "Cmts.User") (width 0.3) (fill none))
@@
   )
   (footprint "eduboardv2:BAT-TH_CR2032-BS-6-1" (layer "F.Cu")
-    (at 89 69 180)
+    (at 86 71 -90)
     (property "JLC Part" "Extended Part")
     (property "LCSC Part" "C70377")
@@
     (property "Sheetname" "UP-Connector, RTC and Flash")
     (attr through_hole)
-    (fp_text reference "B201" (at 0 -4) (layer "F.SilkS")
+    (fp_text reference "B201" (at 0 -4 -270) (layer "F.SilkS")
       (effects (font (size 1 1) (thickness 0.15)))
     )
-    (fp_text value "CR2032-BS-6-1" (at 0 4) (layer "F.Fab")
+    (fp_text value "CR2032-BS-6-1" (at 0 4 -270) (layer "F.Fab")
       (effects (font (size 1 1) (thickness 0.15)))
     )
-    (fp_text user "${REFERENCE}" (at 0 0) (layer "F.Fab")
+    (fp_text user "${REFERENCE}" (at 0 0 -270) (layer "F.Fab")
       (effects (font (size 1 1) (thickness 0.15)))
     )
@@
     (fp_line (start -11.13 8.08) (end 11.13 8.08) (layer "F.SilkS") (width 0.15))
     (fp_circle (center 15.65 -7.95) (end 15.68 -7.95) (layer "F.Fab") (width 0.06) (fill none))
-    (pad "1" smd rect locked (at 14.39 0 180) (size 4.2 3.8) (layers "F.Cu" "F.Paste" "F.Mask")
+    (pad "1" smd rect locked (at 14.39 0 270) (size 4.2 3.8) (layers "F.Cu" "F.Paste" "F.Mask")
       (net 56 "Net-(B201-Pad1)") (pinfunction "1") (pintype "input"))
-    (pad "2" smd rect locked (at -14.39 0 180) (size 4.2 3.8) (layers "F.Cu" "F.Paste" "F.Mask")
+    (pad "2" smd rect locked (at -14.39 0 270) (size 4.2 3.8) (layers "F.Cu" "F.Paste" "F.Mask")
       (net 57 "GND") (pinfunction "2") (pintype "input"))
     (model "${KIPRJMOD}/eduboardv2.3dshapes/BAT-SMD_L28.5-W16.0-H5.5-LS31.3_CR2032-BS-6-1.wrl"
@@
   )
   (footprint "eduboardv2:CONN-TH_3P-P3.81_KF2EDGR-3.81-3P" (layer "F.Cu")
-    (at 71.9675 29.3325 180)
+    (at 70.9675 27.3325 180)
     (property "JLC Part" "Extended Part")
     (property "LCSC Part" "C441183")
@@
   )
   (footprint "eduboardv2:SOIC-8_L5.3-W5.3-P1.27-LS8.0-BL" (layer "F.Cu")
-    (at 88 84 90)
+    (at 72 93 180)
     (property "JLC Part" "Basic Part")
     (property "LCSC Part" "C97521")
@@
     (property "Sheetname" "UP-Connector, RTC and Flash")
     (attr through_hole)
-    (fp_text reference "IC203" (at 0 -7.53 90) (layer "F.SilkS")
+    (fp_text reference "IC203" (at 0 -7.53) (layer "F.SilkS")
       (effects (font (size 1 1) (thickness 0.15)))
     )
-    (fp_text value "W25Q128JVSIQTR" (at 0 7.53 90) (layer "F.Fab")
+    (fp_text value "W25Q128JVSIQTR" (at 0 7.53) (layer "F.Fab")
       (effects (font (size 1 1) (thickness 0.15)))
     )
-    (fp_text user "${REFERENCE}" (at 0 0 90) (layer "F.Fab")
+    (fp_text user "${REFERENCE}" (at 0 0) (layer "F.Fab")
       (effects (font (size 1 1) (thickness 0.15)))
     )
@@
     (fp_circle (center -1.91 4.35) (end -1.76 4.35) (layer "Cmts.User") (width 0.3) (fill none))
     (fp_circle (center -2.59 3.92) (end -2.56 3.92) (layer "F.Fab") (width 0.06) (fill none))
-    (pad "1" smd oval locked (at -1.91 3.53 90) (size 0.63 2.25) (layers "F.Cu" "F.Paste" "F.Mask")
+    (pad "1" smd oval locked (at -1.91 3.53 180) (size 0.63 2.25) (layers "F.Cu" "F.Paste" "F.Mask")
       (net 122 "/UP-Connector, RTC and Flash/FLASH_CS") (pinfunction "CS#") (pintype "unspecified"))
-    (pad "2" smd oval locked (at -0.63 3.53 90) (size 0.63 2.25) (layers "F.Cu" "F.Paste" "F.Mask")
+    (pad "2" smd oval locked (at -0.63 3.53 180) (size 0.63 2.25) (layers "F.Cu" "F.Paste" "F.Mask")
       (net 123 "/UP-Connector, RTC and Flash/SPI0_MISO") (pinfunction "DO") (pintype "unspecified"))
-    (pad "3" smd oval locked (at 0.63 3.53 90) (size 0.63 2.25) (layers "F.Cu" "F.Paste" "F.Mask")
+    (pad "3" smd oval locked (at 0.63 3.53 180) (size 0.63 2.25) (layers "F.Cu" "F.Paste" "F.Mask")
       (net 124 "unconnected-(IC203-Pad3)") (pinfunction "IO2") (pintype "unspecified"))
-    (pad "4" smd oval locked (at 1.9 3.53 90) (size 0.63 2.25) (layers "F.Cu" "F.Paste" "F.Mask")
+    (pad "4" smd oval locked (at 1.9 3.53 180) (size 0.63 2.25) (layers "F.Cu" "F.Paste" "F.Mask")
       (net 57 "GND") (pinfunction "GND") (pintype "unspecified"))
-    (pad "5" smd oval locked (at 1.9 -3.53 90) (size 0.63 2.25) (layers "F.Cu" "F.Paste" "F.Mask")
+    (pad "5" smd oval locked (at 1.9 -3.53 180) (size 0.63 2.25) (layers "F.Cu" "F.Paste" "F.Mask")
       (net 127 "/UP-Connector, RTC and Flash/SPI0_MOSI") (pinfunction "DI") (pintype "unspecified"))
-    (pad "6" smd oval locked (at 0.63 -3.53 90) (size 0.63 2.25) (layers "F.Cu" "F.Paste" "F.Mask")
+    (pad "6" smd oval locked (at 0.63 -3.53 180) (size 0.63 2.25) (layers "F.Cu" "F.Paste" "F.Mask")
       (net 126 "/UP-Connector, RTC and Flash/SPI0_CLK") (pinfunction "CLK") (pintype "unspecified"))
-    (pad "7" smd oval locked (at -0.63 -3.53 90) (size 0.63 2.25) (layers "F.Cu" "F.Paste" "F.Mask")
+    (pad "7" smd oval locked (at -0.63 -3.53 180) (size 0.63 2.25) (layers "F.Cu" "F.Paste" "F.Mask")
       (net 125 "unconnected-(IC203-Pad7)") (pinfunction "IO3") (pintype "unspecified"))
-    (pad "8" smd oval locked (at -1.91 -3.53 90) (size 0.63 2.25) (layers "F.Cu" "F.Paste" "F.Mask")
+    (pad "8" smd oval locked (at -1.91 -3.53 180) (size 0.63 2.25) (layers "F.Cu" "F.Paste" "F.Mask")
       (net 58 "+3.3V") (pinfunction "VCC") (pintype "unspecified"))
     (model "${KIPRJMOD}/eduboardv2.3dshapes/SOIC-8_L5.3-W5.3-H1.9-LS7.9-P1.27.wrl"

Commit message: changed pin types and fixed 3D-positions
Parts:
- moved IC301 123.7 mm to (199.0, 26.0)
- moved IC602 58.0 mm to (181.0, 33.0)
- moved B201 1.00 mm to (86.0, 72.0)
