File: up_rtc_flash.kicad_sch (KiCad schematic)
At the start: 14 parts, among them IC201 PCF8563T_5,518, IC202 W25Q128JVSIQTR, X201 PCIE-52P40H, X202 32.768 kHz, X203 TF-15×15, X204 CR1220-2ZX

Commit message: fix power symbol problem.
Connections:
- net GND: now reaches IC202.4 (GND)
- net GND: now also C201.2, C202.1, C203.1, C204.1, IC201.4 (VSS), X203.6 (VSS), X204.2
- net +3.3V: now reaches C204.2, IC202.8 (VCC)
- net +3.3V: now also C202.2, D201.2 (+), R201.2, R202.2, X203.4 (VDD)
Changed lines of the file:
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@@
     (pin "2")
   )
-  (symbol (lib_name "+3.3V_2") (lib_id "eduboardv2:+3.3V") (at 154.94 177.8 0) (unit 1)
+  (symbol (lib_name "+3.3V_4") (lib_id "eduboardv2:+3.3V") (at 154.94 177.8 0) (unit 1)
     (in_bom yes) (on_board yes) (fields_autoplaced)
     (property "Reference" "#PWR0201" (id 0) (at 154.94 181.61 0)
@@
     (pin "8")
   )
-  (symbol (lib_name "GND_2") (lib_id "eduboardv2:GND") (at 190.5 72.39 0) (unit 1)
+  (symbol (lib_id "eduboardv2:GND") (at 190.5 72.39 0) (unit 1)
     (in_bom yes) (on_board yes) (fields_autoplaced)
     (property "Reference" "#PWR0205" (id 0) (at 190.5 78.74 0)
@@
     (pin "2")
   )
-  (symbol (lib_name "GND_3") (lib_id "eduboardv2:GND") (at 189.23 46.99 0) (unit 1)
+  (symbol (lib_id "eduboardv2:GND") (at 189.23 46.99 0) (unit 1)
     (in_bom yes) (on_board yes) (fields_autoplaced)
     (property "Reference" "#PWR0204" (id 0) (at 189.23 53.34 0)
@@
     (pin "2")
   )
-  (symbol (lib_name "+3.3V_1") (lib_id "eduboardv2:+3.3V") (at 240.03 64.77 0) (unit 1)
+  (symbol (lib_id "eduboardv2:+3.3V") (at 240.03 64.77 0) (unit 1)
     (in_bom yes) (on_board yes) (fields_autoplaced)
     (property "Reference" "#PWR0211" (id 0) (at 240.03 68.58 0)
@@
     (pin "1")
   )
-  (symbol (lib_name "GND_1") (lib_id "eduboardv2:GND") (at 161.29 39.37 0) (unit 1)
+  (symbol (lib_id "eduboardv2:GND") (at 161.29 39.37 0) (unit 1)
     (in_bom yes) (on_board yes) (fields_autoplaced)
     (property "Reference" "#PWR0202" (id 0) (at 161.29 45.72 0)
@@
     (pin "2")
   )
-  (symbol (lib_name "+3.3V_2") (lib_id "eduboardv2:+3.3V") (at 236.22 26.67 0) (unit 1)
+  (symbol (lib_name "+3.3V_3") (lib_id "eduboardv2:+3.3V") (at 236.22 26.67 0) (unit 1)
     (in_bom yes) (on_board yes) (fields_autoplaced)
     (property "Reference" "#PWR0209" (id 0) (at 236.22 30.48 0)
@@
     (pin "1")
   )
-  (symbol (lib_name "GND_5") (lib_id "eduboardv2:GND") (at 240.03 72.39 0) (unit 1)
+  (symbol (lib_id "eduboardv2:GND") (at 240.03 72.39 0) (unit 1)
     (in_bom yes) (on_board yes) (fields_autoplaced)
     (property "Reference" "#PWR0212" (id 0) (at 240.03 78.74 0)
