File: display_ui.kicad_sch (KiCad schematic)
At the start: 67 parts, among them SW2 K2-1102SP-C4SC-04, SW3 K2-1102SP-C4SC-04, SW4 K2-1102SP-C4SC-04, SW5 K2-1102SP-C4SC-04, SW6 PEC11R-4220F-S0012, T1 AO3400A, T2 AO3400A, T3 AO3400A, T4 AO3400A, T5 AO3400A, X5 DFR0649

Commit message: work on layout.
Parts:
- added JP8: SolderJumper_2_Bridged, Jumper:SolderJumper-2_P1.3mm_Bridged_Pad1.0x1.5mm, symbol Jumper:SolderJumper_2_Bridged
- X9: TouchController Datasheet (none) -> https://www.buydisplay.com/download/ic/FT6236-FT6336-FT6436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
Connections:
- net +3.3V: no longer X9.26 (~{RD})
- net AN0: now also JP8.2 (B); no longer C17.2, R13.2
- net WS2812_DOUT: now also D15.4 (DIN), R37.1, T4.3 (D); no longer D15.2 (DOUT)
- new net: C17.2, JP8.1 (A), R13.2
- no-connect marks 22 -> 24
Other:
- note added: "Address: 0x38"
- note added: "Display: ER-TFTM035-6 Touch Controller: FT6236"
- note removed: "https://focuslcds.com/content/FT6236.pdf"
- moved on the sheet: C17
Changed lines of the file:
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@@
   (junction (at 117.475 93.98) (diameter 0) (color 0 0 0 0)
   )
+  (junction (at 147.32 93.98) (diameter 0) (color 0 0 0 0)
+  )
   (junction (at 20.32 167.64) (diameter 0) (color 0 0 0 0)
   )
   (junction (at 167.005 25.4) (diameter 0) (color 0 0 0 0)
   )
+  (junction (at 31.75 97.79) (diameter 0) (color 0 0 0 0)
+  )
   (junction (at 213.36 146.05) (diameter 0) (color 0 0 0 0)
   )
@@
   (junction (at 77.47 97.79) (diameter 0) (color 0 0 0 0)
   )
-  (junction (at 34.29 97.79) (diameter 0) (color 0 0 0 0)
-  )
   (junction (at 81.28 167.64) (diameter 0) (color 0 0 0 0)
   )
@@
   (junction (at 69.85 92.71) (diameter 0) (color 0 0 0 0)
   )
-  (junction (at 255.27 107.95) (diameter 0) (color 0 0 0 0)
-  )
   (junction (at 60.325 167.64) (diameter 0) (color 0 0 0 0)
   )
@@
   (no_connect (at 257.175 90.17))
   (no_connect (at 257.175 85.09))
+  (no_connect (at 120.015 96.52))
   (no_connect (at 257.175 87.63))
   (no_connect (at 257.175 97.79))
@@
   (no_connect (at 257.175 64.77))
   (no_connect (at 257.175 49.53))
+  (no_connect (at 257.175 107.95))
   (no_connect (at 257.175 62.23))
   (no_connect (at 257.175 69.85))
@@
     (stroke (width 0) (type default))
   )
-  (wire (pts (xy 30.48 97.79) (xy 34.29 97.79))
+  (wire (pts (xy 30.48 97.79) (xy 31.75 97.79))
     (stroke (width 0) (type default))
   )
@@
     (stroke (width 0) (type default))
   )
-  (wire (pts (xy 241.935 102.87) (xy 257.175 102.87))
+  (wire (pts (xy 147.32 93.98) (xy 151.765 93.98))
     (stroke (width 0) (type default))
   )
-  (wire (pts (xy 111.76 167.64) (xy 121.285 167.64))
+  (wire (pts (xy 241.935 102.87) (xy 257.175 102.87))
     (stroke (width 0) (type default))
   )
-  (wire (pts (xy 257.175 107.95) (xy 255.27 107.95))
+  (wire (pts (xy 111.76 167.64) (xy 121.285 167.64))
     (stroke (width 0) (type default))
   )
@@
     (stroke (width 0) (type default))
   )
-  (wire (pts (xy 145.415 93.98) (xy 151.765 93.98))
+  (wire (pts (xy 145.415 93.98) (xy 147.32 93.98))
     (stroke (width 0) (type default))
   )
@@
     (stroke (width 0) (type default))
   )
+  (wire (pts (xy 41.275 97.79) (xy 43.18 97.79))
+    (stroke (width 0) (type default))
+  )
   (wire (pts (xy 76.2 55.88) (xy 76.2 57.15))
     (stroke (width 0) (type default))
@@
     (stroke (width 0) (type default))
   )
-  (wire (pts (xy 114.935 96.52) (xy 120.015 96.52))
-    (stroke (width 0) (type default))
-  )
   (wire (pts (xy 241.935 95.25) (xy 257.175 95.25))
     (stroke (width 0) (type default))
@@
     (stroke (width 0) (type default))
   )
+  (wire (pts (xy 147.32 83.185) (xy 147.32 93.98))
+    (stroke (width 0) (type default))
+  )
   (wire (pts (xy 211.455 56.515) (xy 219.71 56.515))
     (stroke (width 0) (type default))
@@
     (stroke (width 0) (type default))
   )
-  (wire (pts (xy 255.27 115.57) (xy 255.27 107.95))
+  (wire (pts (xy 31.75 97.79) (xy 33.655 97.79))
+    (stroke (width 0) (type default))
+  )
+  (wire (pts (xy 255.27 46.99) (xy 255.27 115.57))
     (stroke (width 0) (type default))
   )
@@
     (stroke (width 0) (type default))
   )
-  (wire (pts (xy 34.29 97.79) (xy 34.29 99.06))
+  (wire (pts (xy 144.145 83.185) (xy 147.32 83.185))
+    (stroke (width 0) (type default))
+  )
+  (wire (pts (xy 31.75 97.79) (xy 31.75 99.06))
     (stroke (width 0) (type default))
   )
@@
     (stroke (width 0) (type default))
   )
-  (wire (pts (xy 34.29 97.79) (xy 40.64 97.79))
-    (stroke (width 0) (type default))
-  )
   (wire (pts (xy 241.935 125.73) (xy 257.175 125.73))
     (stroke (width 0) (type default))
@@
     (stroke (width 0) (type default))
   )
-  (wire (pts (xy 34.29 106.68) (xy 34.29 105.41))
+  (wire (pts (xy 31.75 106.68) (xy 31.75 105.41))
     (stroke (width 0) (type default))
   )
@@
     (stroke (width 0) (type default))
   )
-  (wire (pts (xy 255.27 107.95) (xy 255.27 46.99))
-    (stroke (width 0) (type default))
-  )
   (wire (pts (xy 255.27 42.545) (xy 255.27 46.99))
     (stroke (width 0) (type default))
@@
     (effects (font (size 1.27 1.27)) (justify left bottom))
   )
-  (text "https://focuslcds.com/content/FT6236.pdf" (at 233.045 164.465 0)
+  (text "Address:\n0x38" (at 224.155 120.65 0)
+    (effects (font (size 1.27 1.27)) (justify left bottom))
+  )
+  (text "Display: ER-TFTM035-6\n\nTouch Controller: FT6236\n" (at 261.62 153.67 0)
     (effects (font (size 1.27 1.27)) (justify left bottom))
   )
@@
     )
   )
-  (global_label "WS2812_DOUT" (shape output) (at 114.935 96.52 180) (fields_autoplaced)
+  (global_label "WS2812_DOUT" (shape output) (at 144.145 83.185 180) (fields_autoplaced)
     (effects (font (size 1.27 1.27)) (justify right))
-    (property "Intersheetrefs" "${INTERSHEET_REFS}" (at 99.1567 96.4406 0)
+    (property "Intersheetrefs" "${INTERSHEET_REFS}" (at 128.3667 83.1056 0)
       (effects (font (size 1.27 1.27)) (justify right) hide)
     )
@@
     )
   )
-  (global_label "AN0" (shape output) (at 40.64 97.79 0) (fields_autoplaced)
+  (global_label "AN0" (shape output) (at 43.18 97.79 0) (fields_autoplaced)
     (effects (font (size 1.27 1.27)) (justify left))
-    (property "Intersheetrefs" "${INTERSHEET_REFS}" (at 46.6817 97.7106 0)
+    (property "Intersheetrefs" "${INTERSHEET_REFS}" (at 49.2217 97.7106 0)
       (effects (font (size 1.27 1.27)) (justify left) hide)
     )
@@
     )
   )
-  (symbol (lib_id "eduboardv2:GND") (at 34.29 105.41 0) (unit 1)
+  (symbol (lib_id "eduboardv2:GND") (at 31.75 105.41 0) (unit 1)
     (in_bom yes) (on_board yes) (dnp no) (fields_autoplaced)
-    (property "Reference" "#PWR054" (at 34.29 111.76 0)
+    (property "Reference" "#PWR054" (at 31.75 111.76 0)
       (effects (font (size 1.27 1.27)) hide)
     )
-    (property "Value" "GND" (at 34.29 110.49 0)
+    (property "Value" "GND" (at 31.75 110.49 0)
       (effects (font (size 1.27 1.27)))
     )
-    (property "Footprint" "" (at 34.29 105.41 0)
+    (property "Footprint" "" (at 31.75 105.41 0)
       (effects (font (size 1.27 1.27)) hide)
     )
-    (property "Datasheet" "" (at 34.29 105.41 0)
+    (property "Datasheet" "" (at 31.75 105.41 0)
       (effects (font (size 1.27 1.27)) hide)
     )
@@
     )
   )
+  (symbol (lib_id "Jumper:SolderJumper_2_Bridged") (at 37.465 97.79 0) (unit 1)
+    (in_bom yes) (on_board yes) (dnp no)
+    (property "Reference" "JP8" (at 34.29 96.52 0)
+      (effects (font (size 1.27 1.27)))
+    )
+    (property "Value" "SolderJumper_2_Bridged" (at 37.465 95.25 0)
+      (effects (font (size 1.27 1.27)) hide)
+    )
+    (property "Footprint" "Jumper:SolderJumper-2_P1.3mm_Bridged_Pad1.0x1.5mm" (at 37.465 97.79 0)
+      (effects (font (size 1.27 1.27)) hide)
+    )
+    (property "Datasheet" "~" (at 37.465 97.79 0)
+      (effects (font (size 1.27 1.27)) hide)
+    )
+    (pin "1")
+    (pin "2")
+    (instances
+      (project "EduboardV2_Baseboard"
+        (path "/280adf03-05ea-4001-ab24-a5a43e6d4cc9/079bc49e-d545-405c-843f-4b3e915cef08"
+          (reference "JP8") (unit 1)
+        )
+        (path "/280adf03-05ea-4001-ab24-a5a43e6d4cc9/92753037-c50f-47ac-9b4f-72ea899f1ef8"
+          (reference "JP9") (unit 1)
+        )
+      )
+    )
+  )
   (symbol (lib_id "eduboardv2:GND") (at 77.47 113.03 0) (unit 1)
     (in_bom yes) (on_board yes) (dnp no) (fields_autoplaced)
@@
     )
   )
-  (symbol (lib_id "eduboardv2:0402B102K500NT") (at 34.29 102.87 90) (unit 1)
+  (symbol (lib_id "eduboardv2:0402B102K500NT") (at 31.75 102.87 90) (unit 1)
     (in_bom yes) (on_board yes) (dnp no) (fields_autoplaced)
-    (property "Reference" "C17" (at 38.1 101.5999 90)
+    (property "Reference" "C17" (at 35.56 101.5999 90)
       (effects (font (size 1.27 1.27)) (justify right))
     )
-    (property "Value" "1nF" (at 38.1 104.1399 90)
+    (property "Value" "1nF" (at 35.56 104.1399 90)
       (effects (font (size 1.27 1.27)) (justify right))
     )
-    (property "Footprint" "Capacitor_SMD:C_0402_1005Metric_Pad0.74x0.62mm_HandSolder" (at 41.91 102.87 0)
+    (property "Footprint" "Capacitor_SMD:C_0402_1005Metric_Pad0.74x0.62mm_HandSolder" (at 39.37 102.87 0)
       (effects (font (size 1.27 1.27)) hide)
     )
-    (property "Datasheet" "https://lcsc.com/product-detail/Multilayer-Ceramic-Capacitors-MLCC-SMD-SMT_1nF-102-10-50V_C1523.html" (at 46.99 102.87 0)
+    (property "Datasheet" "https://lcsc.com/product-detail/Multilayer-Ceramic-Capacitors-MLCC-SMD-SMT_1nF-102-10-50V_C1523.html" (at 44.45 102.87 0)
       (effects (font (size 1.27 1.27)) hide)
     )
-    (property "Manufacturer" "FH" (at 49.53 102.87 0)
+    (property "Manufacturer" "FH" (at 46.99 102.87 0)
       (effects (font (size 1.27 1.27)) hide)
     )
-    (property "LCSC Part" "C1523" (at 52.07 102.87 0)
+    (property "LCSC Part" "C1523" (at 49.53 102.87 0)
       (effects (font (size 1.27 1.27)) hide)
     )
-    (property "JLC Part" "Basic Part" (at 54.61 102.87 0)
+    (property "JLC Part" "Basic Part" (at 52.07 102.87 0)
       (effects (font (size 1.27 1.27)) hide)
     )
-    (property "MPN" "0402B102K500NT" (at 39.37 102.87 0)
+    (property "MPN" "0402B102K500NT" (at 36.83 102.87 0)
       (effects (font (size 1.27 1.27)) hide)
     )
@@
       (effects (font (size 1.27 1.27)) hide)
     )
-    (property "Datasheet" "" (at 266.7 53.34 0)
+    (property "Datasheet" "https://www.buydisplay.com/lcd-3-5-inch-320x480-tft-display-module-optl-touch-screen-w-breakout-board" (at 266.7 53.34 0)
+      (effects (font (size 1.27 1.27)) hide)
+    )
+    (property "TouchController Datasheet" "https://www.buydisplay.com/download/ic/FT6236-FT6336-FT6436L-FT6436_Datasheet.pdf" (at 270.51 89.535 0)
       (effects (font (size 1.27 1.27)) hide)
     )

Commit message: layout done so far. Have to check everything again
Parts:
- R13: JLC Part (none) -> Extended Part
- X5: now left out of the parts list
- X9: value ~ -> BH-00105; JLC Part (none) -> Extended Part; LCSC Part (none) -> C2685092
Changed lines of the file:
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@@
   )
   (symbol (lib_id "EduboardV2_kicadlib:DFR0649") (at 230.505 55.245 0) (unit 1)
-    (in_bom yes) (on_board yes) (dnp no)
+    (in_bom no) (on_board yes) (dnp no)
     (property "Reference" "X5" (at 222.25 43.18 0)
       (effects (font (size 1.27 1.27)) (justify left))
@@
       (effects (font (size 1.27 1.27)) hide)
     )
+    (property "JLC Part" "Extended Part" (at 25.4 97.79 0)
+      (effects (font (size 1.27 1.27)) hide)
+    )
     (pin "1")
     (pin "2")
@@
       (effects (font (size 1.27 1.27)) (justify left))
     )
-    (property "Value" "~" (at 266.7 53.34 0)
+    (property "Value" "BH-00105" (at 273.05 88.9 0)
       (effects (font (size 1.27 1.27)))
     )
@@
       (effects (font (size 1.27 1.27)) hide)
     )
+    (property "LCSC Part" "C2685092" (at 270.51 89.535 0)
+      (effects (font (size 1.27 1.27)) hide)
+    )
+    (property "JLC Part" "Extended Part" (at 270.51 89.535 0)
+      (effects (font (size 1.27 1.27)) hide)
+    )
